File: H-Bridge.sch (KiCad schematic (older format))
At the start: 66 parts

Commit message: デッドタイム挿入回路を削除、マイコンブロック作成
Parts:
- removed C? (x4): 10n, symbol Device:C_Small
- removed C? (x2): 0.1u, symbol Device:C_Small
- removed D? (x4): D_Schottky_Small, symbol Device:D_Schottky_Small
- removed R? (x4): 0, symbol Device:R_Small
- removed R? (x4): 10, symbol Device:R_Small
- removed U? (x12): 74HC14, symbol 74xx:74HC14
Connections:
- net labels added: GATE_AN, GATE_AP, GATE_BN, GATE_BP
- net labels removed: +3.3V, GateA, GateB
- wire segments 188 -> 122
Other:
- moved on the sheet: C?, D?, Q?, R?, U?

Commit message: 第１版回路図完成
Parts:
- gave numbers to parts that had none: 36

Commit message: フットプリント割り付け＆Netリスト出力
Parts:
- C13, C14, C15, C16, C17, C18: footprint (none) -> Capacitors_SMD:C_0603_HandSoldering
- D10, D11, D8, D9: footprint (none) -> Diodes_SMD:D_SMA_Handsoldering
- D6, D7: footprint (none) -> Diodes_SMD:D_TUMD2
- Q1, Q2, Q3, Q4: footprint (none) -> TO_SOT_Packages_THT:TO-220-3_Horizontal_Reversed
- R13, R14, R15, R16, R17, R18, R19, R20, R25, R26, R27, R28: footprint (none) -> Resistors_SMD:R_0603_HandSoldering
- R21, R22, R23, R24: footprint (none) -> Resistors_SMD:R_0805_HandSoldering
- U5, U6, U7, U8: footprint (none) -> Housings_SOIC:SO-5_4.4x3.6mm_Pitch1.27mm
Changed lines of the file:
@@
 F 0 "U5" H 4900 2125 50  0000 C CNN
 F 1 "TLP152" H 4900 2034 50  0000 C CNN
-F 2 "" H 4900 1600 50  0001 C CNN
+F 2 "Housings_SOIC:SO-5_4.4x3.6mm_Pitch1.27mm" H 4900 1600 50  0001 C CNN
 F 3 "" H 4900 1600 50  0001 C CNN
 	1    4900 1600
@@
 F 0 "Q1" H 7355 1646 50  0000 L CNN
 F 1 "Q_NMOS_GDS" H 7355 1555 50  0000 L CNN
-F 2 "" H 7350 1700 50  0001 C CNN
+F 2 "TO_SOT_Packages_THT:TO-220-3_Horizontal_Reversed" H 7350 1700 50  0001 C CNN
 F 3 "~" H 7150 1600 50  0001 C CNN
 	1    7150 1600
@@
 F 0 "D8" V 7954 1679 50  0000 L CNN
 F 1 "D" V 8045 1679 50  0000 L CNN
-F 2 "" H 8000 1600 50  0001 C CNN
+F 2 "Diodes_SMD:D_SMA_Handsoldering" H 8000 1600 50  0001 C CNN
 F 3 "~" H 8000 1600 50  0001 C CNN
 	1    8000 1600
@@
 F 0 "D6" V 5946 1021 50  0000 R CNN
 F 1 "D" V 5855 1021 50  0000 R CNN
-F 2 "" H 5900 1100 50  0001 C CNN
+F 2 "Diodes_SMD:D_TUMD2" H 5900 1100 50  0001 C CNN
 F 3 "~" H 5900 1100 50  0001 C CNN
 	1    5900 1100
@@
 F 0 "C13" H 5592 1496 50  0000 L CNN
 F 1 "0.1u" H 5592 1405 50  0000 L CNN
-F 2 "" H 5500 1450 50  0001 C CNN
+F 2 "Capacitors_SMD:C_0603_HandSoldering" H 5500 1450 50  0001 C CNN
 F 3 "~" H 5500 1450 50  0001 C CNN
 	1    5500 1450
@@
 F 0 "C17" H 5991 1496 50  0000 L CNN
 F 1 "10u" H 5991 1405 50  0000 L CNN
-F 2 "" H 5900 1450 50  0001 C CNN
+F 2 "Capacitors_SMD:C_0603_HandSoldering" H 5900 1450 50  0001 C CNN
 F 3 "~" H 5900 1450 50  0001 C CNN
 	1    5900 1450
@@
 F 0 "R21" V 6104 1600 50  0000 C CNN
 F 1 "4.7" V 6195 1600 50  0000 C CNN
-F 2 "" H 6300 1600 50  0001 C CNN
+F 2 "Resistors_SMD:R_0805_HandSoldering" H 6300 1600 50  0001 C CNN
 F 3 "~" H 6300 1600 50  0001 C CNN
 	1    6300 1600
@@
 F 0 "R25" H 6709 1796 50  0000 L CNN
 F 1 "10k" H 6709 1705 50  0000 L CNN
-F 2 "" H 6650 1750 50  0001 C CNN
+F 2 "Resistors_SMD:R_0603_HandSoldering" H 6650 1750 50  0001 C CNN
 F 3 "~" H 6650 1750 50  0001 C CNN
 	1    6650 1750
@@
 F 0 "R13" V 3804 1300 50  0000 C CNN
 F 1 "200" V 3895 1300 50  0000 C CNN
-F 2 "" H 4000 1300 50  0001 C CNN
+F 2 "Resistors_SMD:R_0603_HandSoldering" H 4000 1300 50  0001 C CNN
 F 3 "~" H 4000 1300 50  0001 C CNN
 	1    4000 1300
@@
 F 0 "R17" H 4241 1646 50  0000 R CNN
 F 1 "10k" H 4241 1555 50  0000 R CNN
-F 2 "" H 4300 1600 50  0001 C CNN
+F 2 "Resistors_SMD:R_0603_HandSoldering" H 4300 1600 50  0001 C CNN
 F 3 "~" H 4300 1600 50  0001 C CNN
 	1    4300 1600
@@
 F 0 "U6" H 4900 3325 50  0000 C CNN
 F 1 "TLP152" H 4900 3234 50  0000 C CNN
-F 2 "" H 4900 2800 50  0001 C CNN
+F 2 "Housings_SOIC:SO-5_4.4x3.6mm_Pitch1.27mm" H 4900 2800 50  0001 C CNN
 F 3 "" H 4900 2800 50  0001 C CNN
 	1    4900 2800
@@
 F 0 "Q2" H 7355 2846 50  0000 L CNN
 F 1 "Q_NMOS_GDS" H 7355 2755 50  0000 L CNN
-F 2 "" H 7350 2900 50  0001 C CNN
+F 2 "TO_SOT_Packages_THT:TO-220-3_Horizontal_Reversed" H 7350 2900 50  0001 C CNN
 F 3 "~" H 7150 2800 50  0001 C CNN
 	1    7150 2800
@@
 F 0 "D9" V 7954 2879 50  0000 L CNN
 F 1 "D" V 8045 2879 50  0000 L CNN
-F 2 "" H 8000 2800 50  0001 C CNN
+F 2 "Diodes_SMD:D_SMA_Handsoldering" H 8000 2800 50  0001 C CNN
 F 3 "~" H 8000 2800 50  0001 C CNN
 	1    8000 2800
@@
 F 0 "C14" H 5592 2696 50  0000 L CNN
 F 1 "0.1u" H 5592 2605 50  0000 L CNN
-F 2 "" H 5500 2650 50  0001 C CNN
+F 2 "Capacitors_SMD:C_0603_HandSoldering" H 5500 2650 50  0001 C CNN
 F 3 "~" H 5500 2650 50  0001 C CNN
 	1    5500 2650
@@
 F 0 "R22" V 6104 2800 50  0000 C CNN
 F 1 "4.7" V 6195 2800 50  0000 C CNN
-F 2 "" H 6300 2800 50  0001 C CNN
+F 2 "Resistors_SMD:R_0805_HandSoldering" H 6300 2800 50  0001 C CNN
 F 3 "~" H 6300 2800 50  0001 C CNN
 	1    6300 2800
@@
 F 0 "R26" H 6709 2996 50  0000 L CNN
 F 1 "10k" H 6709 2905 50  0000 L CNN
-F 2 "" H 6650 2950 50  0001 C CNN
+F 2 "Resistors_SMD:R_0603_HandSoldering" H 6650 2950 50  0001 C CNN
 F 3 "~" H 6650 2950 50  0001 C CNN
 	1    6650 2950
@@
 F 0 "R14" V 3804 2500 50  0000 C CNN
 F 1 "200" V 3895 2500 50  0000 C CNN
-F 2 "" H 4000 2500 50  0001 C CNN
+F 2 "Resistors_SMD:R_0603_HandSoldering" H 4000 2500 50  0001 C CNN
 F 3 "~" H 4000 2500 50  0001 C CNN
 	1    4000 2500
@@
 F 0 "R18" H 4241 2846 50  0000 R CNN
 F 1 "10k" H 4241 2755 50  0000 R CNN
-F 2 "" H 4300 2800 50  0001 C CNN
+F 2 "Resistors_SMD:R_0603_HandSoldering" H 4300 2800 50  0001 C CNN
 F 3 "~" H 4300 2800 50  0001 C CNN
 	1    4300 2800
@@
 F 0 "U7" H 4900 5025 50  0000 C CNN
 F 1 "TLP152" H 4900 4934 50  0000 C CNN
-F 2 "" H 4900 4500 50  0001 C CNN
+F 2 "Housings_SOIC:SO-5_4.4x3.6mm_Pitch1.27mm" H 4900 4500 50  0001 C CNN
 F 3 "" H 4900 4500 50  0001 C CNN
 	1    4900 4500
@@
 F 0 "Q3" H 7355 4546 50  0000 L CNN
 F 1 "Q_NMOS_GDS" H 7355 4455 50  0000 L CNN
-F 2 "" H 7350 4600 50  0001 C CNN
+F 2 "TO_SOT_Packages_THT:TO-220-3_Horizontal_Reversed" H 7350 4600 50  0001 C CNN
 F 3 "~" H 7150 4500 50  0001 C CNN
 	1    7150 4500
@@
 F 0 "D10" V 7954 4579 50  0000 L CNN
 F 1 "D" V 8045 4579 50  0000 L CNN
-F 2 "" H 8000 4500 50  0001 C CNN
+F 2 "Diodes_SMD:D_SMA_Handsoldering" H 8000 4500 50  0001 C CNN
 F 3 "~" H 8000 4500 50  0001 C CNN
 	1    8000 4500
@@
 F 0 "D7" V 5946 3921 50  0000 R CNN
 F 1 "D" V 5855 3921 50  0000 R CNN
-F 2 "" H 5900 4000 50  0001 C CNN
+F 2 "Diodes_SMD:D_TUMD2" H 5900 4000 50  0001 C CNN
 F 3 "~" H 5900 4000 50  0001 C CNN
 	1    5900 4000
@@
 F 0 "C15" H 5592 4396 50  0000 L CNN
 F 1 "0.1u" H 5592 4305 50  0000 L CNN
-F 2 "" H 5500 4350 50  0001 C CNN
+F 2 "Capacitors_SMD:C_0603_HandSoldering" H 5500 4350 50  0001 C CNN
 F 3 "~" H 5500 4350 50  0001 C CNN
 	1    5500 4350
@@
 F 0 "C18" H 5991 4396 50  0000 L CNN
 F 1 "10u" H 5991 4305 50  0000 L CNN
-F 2 "" H 5900 4350 50  0001 C CNN
+F 2 "Capacitors_SMD:C_0603_HandSoldering" H 5900 4350 50  0001 C CNN
 F 3 "~" H 5900 4350 50  0001 C CNN
 	1    5900 4350
@@
 F 0 "R23" V 6104 4500 50  0000 C CNN
 F 1 "4.7" V 6195 4500 50  0000 C CNN
-F 2 "" H 6300 4500 50  0001 C CNN
+F 2 "Resistors_SMD:R_0805_HandSoldering" H 6300 4500 50  0001 C CNN
 F 3 "~" H 6300 4500 50  0001 C CNN
 	1    6300 4500
@@
 F 0 "R27" H 6709 4696 50  0000 L CNN
 F 1 "10k" H 6709 4605 50  0000 L CNN
-F 2 "" H 6650 4650 50  0001 C CNN
+F 2 "Resistors_SMD:R_0603_HandSoldering" H 6650 4650 50  0001 C CNN
 F 3 "~" H 6650 4650 50  0001 C CNN
 	1    6650 4650
@@
 F 0 "R15" V 3804 4200 50  0000 C CNN
 F 1 "200" V 3895 4200 50  0000 C CNN
-F 2 "" H 4000 4200 50  0001 C CNN
+F 2 "Resistors_SMD:R_0603_HandSoldering" H 4000 4200 50  0001 C CNN
 F 3 "~" H 4000 4200 50  0001 C CNN
 	1    4000 4200
@@
 F 0 "R19" H 4241 4546 50  0000 R CNN
 F 1 "10k" H 4241 4455 50  0000 R CNN
-F 2 "" H 4300 4500 50  0001 C CNN
+F 2 "Resistors_SMD:R_0603_HandSoldering" H 4300 4500 50  0001 C CNN
 F 3 "~" H 4300 4500 50  0001 C CNN
 	1    4300 4500
@@
 F 0 "U8" H 4900 6225 50  0000 C CNN
 F 1 "TLP152" H 4900 6134 50  0000 C CNN
-F 2 "" H 4900 5700 50  0001 C CNN
+F 2 "Housings_SOIC:SO-5_4.4x3.6mm_Pitch1.27mm" H 4900 5700 50  0001 C CNN
 F 3 "" H 4900 5700 50  0001 C CNN
 	1    4900 5700
@@
 F 0 "Q4" H 7355 5746 50  0000 L CNN
 F 1 "Q_NMOS_GDS" H 7355 5655 50  0000 L CNN
-F 2 "" H 7350 5800 50  0001 C CNN
+F 2 "TO_SOT_Packages_THT:TO-220-3_Horizontal_Reversed" H 7350 5800 50  0001 C CNN
 F 3 "~" H 7150 5700 50  0001 C CNN
 	1    7150 5700
@@
 F 0 "D11" V 7954 5779 50  0000 L CNN
 F 1 "D" V 8045 5779 50  0000 L CNN
-F 2 "" H 8000 5700 50  0001 C CNN
+F 2 "Diodes_SMD:D_SMA_Handsoldering" H 8000 5700 50  0001 C CNN
 F 3 "~" H 8000 5700 50  0001 C CNN
 	1    8000 5700
@@
 F 0 "C16" H 5592 5596 50  0000 L CNN
 F 1 "0.1u" H 5592 5505 50  0000 L CNN
-F 2 "" H 5500 5550 50  0001 C CNN
+F 2 "Capacitors_SMD:C_0603_HandSoldering" H 5500 5550 50  0001 C CNN
 F 3 "~" H 5500 5550 50  0001 C CNN
 	1    5500 5550
@@
 F 0 "R24" V 6104 5700 50  0000 C CNN
 F 1 "4.7" V 6195 5700 50  0000 C CNN
-F 2 "" H 6300 5700 50  0001 C CNN
+F 2 "Resistors_SMD:R_0805_HandSoldering" H 6300 5700 50  0001 C CNN
 F 3 "~" H 6300 5700 50  0001 C CNN
 	1    6300 5700
@@
 F 0 "R28" H 6709 5896 50  0000 L CNN
 F 1 "10k" H 6709 5805 50  0000 L CNN
-F 2 "" H 6650 5850 50  0001 C CNN
+F 2 "Resistors_SMD:R_0603_HandSoldering" H 6650 5850 50  0001 C CNN
 F 3 "~" H 6650 5850 50  0001 C CNN
 	1    6650 5850
@@
 F 0 "R16" V 3804 5400 50  0000 C CNN
 F 1 "200" V 3895 5400 50  0000 C CNN
-F 2 "" H 4000 5400 50  0001 C CNN
+F 2 "Resistors_SMD:R_0603_HandSoldering" H 4000 5400 50  0001 C CNN
 F 3 "~" H 4000 5400 50  0001 C CNN
 	1    4000 5400
@@
 F 0 "R20" H 4241 5746 50  0000 R CNN
 F 1 "10k" H 4241 5655 50  0000 R CNN
-F 2 "" H 4300 5700 50  0001 C CNN
+F 2 "Resistors_SMD:R_0603_HandSoldering" H 4300 5700 50  0001 C CNN
 F 3 "~" H 4300 5700 50  0001 C CNN
 	1    4300 5700

Commit message: フライホイールダイオード交換
Parts:
- D10, D11, D8, D9: footprint Diodes_SMD:D_SMA_Handsoldering -> Diodes_SMD:D_SMB
Changed lines of the file:
@@
 F 0 "D8" V 7954 1679 50  0000 L CNN
 F 1 "D" V 8045 1679 50  0000 L CNN
-F 2 "Diodes_SMD:D_SMA_Handsoldering" H 8000 1600 50  0001 C CNN
+F 2 "Diodes_SMD:D_SMB" H 8000 1600 50  0001 C CNN
 F 3 "~" H 8000 1600 50  0001 C CNN
 	1    8000 1600
@@
 F 0 "D9" V 7954 2879 50  0000 L CNN
 F 1 "D" V 8045 2879 50  0000 L CNN
-F 2 "Diodes_SMD:D_SMA_Handsoldering" H 8000 2800 50  0001 C CNN
+F 2 "Diodes_SMD:D_SMB" H 8000 2800 50  0001 C CNN
 F 3 "~" H 8000 2800 50  0001 C CNN
 	1    8000 2800
@@
 F 0 "D10" V 7954 4579 50  0000 L CNN
 F 1 "D" V 8045 4579 50  0000 L CNN
-F 2 "Diodes_SMD:D_SMA_Handsoldering" H 8000 4500 50  0001 C CNN
+F 2 "Diodes_SMD:D_SMB" H 8000 4500 50  0001 C CNN
 F 3 "~" H 8000 4500 50  0001 C CNN
 	1    8000 4500
@@
 F 0 "D11" V 7954 5779 50  0000 L CNN
 F 1 "D" V 8045 5779 50  0000 L CNN
-F 2 "Diodes_SMD:D_SMA_Handsoldering" H 8000 5700 50  0001 C CNN
+F 2 "Diodes_SMD:D_SMB" H 8000 5700 50  0001 C CNN
 F 3 "~" H 8000 5700 50  0001 C CNN
 	1    8000 5700

Commit message: kicadバージョン更新
Parts:
- U5, U6, U7, U8: symbol mylib:TLP152 -> spindleMD_v2-rescue:TLP152-mylib
Changed lines of the file:
@@
 EESchema Schematic File Version 4
 LIBS:spindleMD_v2-cache
-EELAYER 26 0
+EELAYER 29 0
 EELAYER END
 $Descr A4 11693 8268
@@
 $EndDescr
 $Comp
-L mylib:TLP152 U5
+L spindleMD_v2-rescue:TLP152-mylib U5
 U 1 1 5C7B8F53
 P 4900 1600
@@
 	5900 850  5900 950
 $Comp
-L mylib:TLP152 U6
+L spindleMD_v2-rescue:TLP152-mylib U6
 U 1 1 5C7BBD60
 P 4900 2800
@@
 Connection ~ 7250 1300
 $Comp
-L mylib:TLP152 U7
+L spindleMD_v2-rescue:TLP152-mylib U7
 U 1 1 5C7C69E1
 P 4900 4500
@@
 	5900 3750 5900 3850
 $Comp
-L mylib:TLP152 U8
+L spindleMD_v2-rescue:TLP152-mylib U8
 U 1 1 5C7C6A55
 P 4900 5700
