File: VoltageSensing.sch (KiCad schematic (older format))
At the start: 10 parts

Commit message: 第１版回路図完成
Parts:
- gave numbers to parts that had none: 10

Commit message: フットプリント割り付け＆Netリスト出力
Parts:
- C20, C21, C22, C23: footprint (none) -> Capacitors_SMD:C_0603_HandSoldering
- R29, R30, R31, R32, R33: footprint (none) -> Resistors_SMD:R_0603_HandSoldering
- U10: footprint (none) -> Housings_SSOP:QSOP-16_3.9x4.9mm_Pitch0.635mm
Changed lines of the file:
@@
 F 0 "U10" H 5550 4550 50  0000 C CNN
 F 1 "ADuM3190" H 5550 4450 50  0000 C CNN
-F 2 "" H 5550 3650 50  0001 C CNN
+F 2 "Housings_SSOP:QSOP-16_3.9x4.9mm_Pitch0.635mm" H 5550 3650 50  0001 C CNN
 F 3 "" H 5550 3650 50  0001 C CNN
 	1    5550 3650
@@
 F 0 "R29" V 4004 3750 50  0000 C CNN
 F 1 "10k" V 4095 3750 50  0000 C CNN
-F 2 "" H 4200 3750 50  0001 C CNN
+F 2 "Resistors_SMD:R_0603_HandSoldering" H 4200 3750 50  0001 C CNN
 F 3 "~" H 4200 3750 50  0001 C CNN
 	1    4200 3750
@@
 F 0 "R33" V 8043 3850 50  0000 C CNN
 F 1 "100k" V 8134 3850 50  0000 C CNN
-F 2 "" V 8180 3850 50  0001 C CNN
+F 2 "Resistors_SMD:R_0603_HandSoldering" V 8180 3850 50  0001 C CNN
 F 3 "~" H 8250 3850 50  0001 C CNN
 	1    8250 3850
@@
 F 0 "R32" H 7970 4146 50  0000 L CNN
 F 1 "1k" H 7970 4055 50  0000 L CNN
-F 2 "" V 7830 4100 50  0001 C CNN
+F 2 "Resistors_SMD:R_0603_HandSoldering" V 7830 4100 50  0001 C CNN
 F 3 "~" H 7900 4100 50  0001 C CNN
 	1    7900 4100
@@
 F 0 "R31" V 7343 3850 50  0000 C CNN
 F 1 "100k" V 7434 3850 50  0000 C CNN
-F 2 "" V 7480 3850 50  0001 C CNN
+F 2 "Resistors_SMD:R_0603_HandSoldering" V 7480 3850 50  0001 C CNN
 F 3 "~" H 7550 3850 50  0001 C CNN
 	1    7550 3850
@@
 F 0 "R30" V 6750 4050 50  0000 C CNN
 F 1 "100k" V 6850 4050 50  0000 C CNN
-F 2 "" V 6880 4050 50  0001 C CNN
+F 2 "Resistors_SMD:R_0603_HandSoldering" V 6880 4050 50  0001 C CNN
 F 3 "~" H 6950 4050 50  0001 C CNN
 	1    6950 4050
@@
 F 0 "C23" V 6771 3250 50  0000 C CNN
 F 1 "1u" V 6862 3250 50  0000 C CNN
-F 2 "" H 7000 3250 50  0001 C CNN
+F 2 "Capacitors_SMD:C_0603_HandSoldering" H 7000 3250 50  0001 C CNN
 F 3 "~" H 7000 3250 50  0001 C CNN
 	1    7000 3250
@@
 F 0 "C20" V 4429 3350 50  0000 C CNN
 F 1 "1u" V 4338 3350 50  0000 C CNN
-F 2 "" H 4200 3350 50  0001 C CNN
+F 2 "Capacitors_SMD:C_0603_HandSoldering" H 4200 3350 50  0001 C CNN
 F 3 "~" H 4200 3350 50  0001 C CNN
 	1    4200 3350
@@
 F 0 "C22" V 5921 2700 50  0000 C CNN
 F 1 "1u" V 6012 2700 50  0000 C CNN
-F 2 "" H 6150 2700 50  0001 C CNN
+F 2 "Capacitors_SMD:C_0603_HandSoldering" H 6150 2700 50  0001 C CNN
 F 3 "~" H 6150 2700 50  0001 C CNN
 	1    6150 2700
@@
 F 0 "C21" V 5129 2700 50  0000 C CNN
 F 1 "1u" V 5038 2700 50  0000 C CNN
-F 2 "" H 4900 2700 50  0001 C CNN
+F 2 "Capacitors_SMD:C_0603_HandSoldering" H 4900 2700 50  0001 C CNN
 F 3 "~" H 4900 2700 50  0001 C CNN
 	1    4900 2700

Commit message: kicadバージョン更新
Parts:
- U10: symbol mylib:ADuM3190 -> spindleMD_v2-rescue:ADuM3190-mylib
Changed lines of the file:
@@
 EESchema Schematic File Version 4
 LIBS:spindleMD_v2-cache
-EELAYER 26 0
+EELAYER 29 0
 EELAYER END
 $Descr A4 11693 8268
@@
 $EndDescr
 $Comp
-L mylib:ADuM3190 U10
+L spindleMD_v2-rescue:ADuM3190-mylib U10
 U 1 1 5C78FD61
 P 5550 3650
